File: tanklevel.kicad_sch (KiCad schematic)
At the start: 71 parts, among them J1 Conn_01x02_Socket, J2 Conn_01x02_Socket, J3 RJ45_Amphenol_RJMG1BD3B8K1ANR, U1 wuerthDebug6, U2 MCP6022, U3 MCP6022, U4 R-78E3.3-0.5, U5 KSZ8081MLX, U6 ESP32-WROOM-32, U7 MCP3221

Commit message: feat: Switch back to LAN8720A
Parts:
- removed C10, C16: 22u, Capacitor_SMD:C_0805_2012Metric_Pad1.18x1.45mm_HandSolder, symbol Device:C
- removed C11, C14, C8: 100n, Capacitor_SMD:C_0402_1005Metric_Pad0.74x0.62mm_HandSolder, symbol Device:C
- removed C15: 2u2, Capacitor_SMD:C_0603_1608Metric_Pad1.08x0.95mm_HandSolder, symbol Device:C
- removed C18: 20n, Capacitor_SMD:C_0402_1005Metric_Pad0.74x0.62mm_HandSolder, symbol Device:C
- removed FB1: BLM18KG331SH1D, Capacitor_SMD:C_0603_1608Metric_Pad1.08x0.95mm_HandSolder, symbol Device:FerriteBead_Small
- removed J1, J2: Conn_01x02_Socket, awesome:WAGO2604-1102, symbol Connector:Conn_01x02_Socket
- removed J3: RJ45_Amphenol_RJMG1BD3B8K1ANR, Connector_RJ:RJ45_Amphenol_RJMG1BD3B8K1ANR, symbol Connector:RJ45_Amphenol_RJMG1BD3B8K1ANR
- removed R10, R11: 220R, Resistor_SMD:R_0402_1005Metric_Pad0.72x0.64mm_HandSolder, symbol Device:R
- removed R16, R19, R2: 33R, Resistor_SMD:R_0402_1005Metric_Pad0.72x0.64mm_HandSolder, symbol Device:R
- removed R20, R21, R22, R23: 50R, Resistor_SMD:R_0402_1005Metric_Pad0.72x0.64mm_HandSolder, symbol Device:R
- removed R35: 10K, Resistor_SMD:R_0402_1005Metric_Pad0.72x0.64mm_HandSolder, symbol Device:R
- removed R8, R9: 4K7, Resistor_SMD:R_0402_1005Metric_Pad0.72x0.64mm_HandSolder, symbol Device:R
- removed U3: MCP6022, Package_SO:SOIC-8_3.9x4.9mm_P1.27mm, symbol Amplifier_Operational:MCP6022
- removed U5: KSZ8081MLX, Package_QFP:LQFP-48_7x7mm_P0.5mm, symbol Interface_Ethernet:KSZ8081MLX
- added C17, C19, C21: 100n, Capacitor_SMD:C_0603_1608Metric_Pad1.08x0.95mm_HandSolder, symbol Device:C
- added C28: 470p, Capacitor_SMD:C_0603_1608Metric_Pad1.08x0.95mm_HandSolder, symbol Device:C
- added C29: 1u, Capacitor_SMD:C_0603_1608Metric_Pad1.08x0.95mm_HandSolder, symbol Device:C
- added C30: 20n, Capacitor_SMD:C_0603_1608Metric_Pad1.08x0.95mm_HandSolder, symbol Device:C
- added FB2: BLM18KG331SH1D, Capacitor_SMD:C_0603_1608Metric_Pad1.08x0.95mm_HandSolder, symbol Device:FerriteBead_Small
- added J1: RJ45_Amphenol_RJMG1BD3B8K1ANR, Connector_RJ:RJ45_Amphenol_RJMG1BD3B8K1ANR, symbol Connector:RJ45_Amphenol_RJMG1BD3B8K1ANR
- added J4: WAGO250-204, awesome:WAGO250-204, symbol awesome:WAGO250-204
- added R26, R36, R40, R43: 10K, Resistor_SMD:R_0603_1608Metric_Pad0.98x0.95mm_HandSolder, symbol Device:R
- added R27, R29, R30, R31: 100R, Resistor_SMD:R_0603_1608Metric_Pad0.98x0.95mm_HandSolder, symbol Device:R
- added R32, R33, R34: 33R, Resistor_SMD:R_0603_1608Metric_Pad0.98x0.95mm_HandSolder, symbol Device:R
- added R37: 12K1 1%, Resistor_SMD:R_0603_1608Metric_Pad0.98x0.95mm_HandSolder, symbol Device:R
- added R38, R39, R41, R42: 50R, Resistor_SMD:R_0603_1608Metric_Pad0.98x0.95mm_HandSolder, symbol Device:R
- added R44, R45: 1K, Resistor_SMD:R_0603_1608Metric_Pad0.98x0.95mm_HandSolder, symbol Device:R
- added unit 1 of U2
- added U3: wuerthJTAG, awesome:wuerthJTAG, symbol awesome:wuerthJTAG
- added U5: LAN8720A, Package_DFN_QFN:QFN-24-1EP_4x4mm_P0.5mm_EP2.6x2.6mm, symbol Interface_Ethernet:LAN8720A
- C1, C13, C24, C25, C4, C6: footprint Capacitor_SMD:C_0402_1005Metric_Pad0.74x0.62mm_HandSolder -> Capacitor_SMD:C_0603_1608Metric_Pad1.08x0.95mm_HandSolder
- C7: value 100n -> 1u; footprint Capacitor_SMD:C_0402_1005Metric_Pad0.74x0.62mm_HandSolder -> Capacitor_SMD:C_0603_1608Metric_Pad1.08x0.95mm_HandSolder
- F1, F2: footprint (none) -> Fuse:Fuse_0603_1608Metric_Pad1.05x0.95mm_HandSolder
- PGAIN1: renamed from PGAIN; value 10k -> 3k; footprint (none) -> Potentiometer_THT:Potentiometer_Bourns_3296W_Vertical
- PZERO1: renamed from PZERO; footprint (none) -> Potentiometer_THT:Potentiometer_Bourns_3296W_Vertical
- R1: footprint (none) -> Resistor_SMD:R_1206_3216Metric_Pad1.30x1.75mm_HandSolder; symbol Device:R_Shunt -> Device:R
- R12, R13, R14, R15, R17, R18, R24, R25, R28, R3, R4, R5, R6, R7: footprint Resistor_SMD:R_0402_1005Metric_Pad0.72x0.64mm_HandSolder -> Resistor_SMD:R_0603_1608Metric_Pad0.98x0.95mm_HandSolder
- U2: footprint (none) -> Package_SO:SOIC-8_3.9x4.9mm_P1.27mm
Connections:
- net +3.3V: now also FB2.2, R36.2, U3.1 (VCC)
- net 24V: now also J4.2; no longer D4.1 (A1), F1.1
- net CRS: now also U5.11 (CRS_DV/MODE2)
- net ETHCLK_50M: now also R32.2, U5.5 (XTAL1/CLKIN)
- net GND: now also C7.2, R1.2, C17.2, C19.2, C21.2, C28.1, C29.1, C30.2, J1.R8, J1.SH, J4.3, R26.1, R37.2, R40.2, R43.1, R44.2, R45.2, U3.6 (GND), U5.25 (VSS); no longer C7.1, R1.4, U6.14 (IO12)
- net MDC: now also U5.13 (MDC)
- net MDIO: now also U5.12 (MDIO)
- net NRST: now also U5.15 (RST)
- net RXD0: now also R33.1
- net RXD1: now also R34.1
- net TXD0: now also U5.17 (TXD0)
- net TXD1: now also U5.18 (TXD1)
- net VDDA: now also C7.1, C17.1, C19.1, C21.1, C30.1, FB2.1, J1.R4 (TCT), J1.R5 (RCT), R38.1, R39.1, R41.1, R42.1, U5.1 (VDD2A), U5.19 (VDD1A), U5.9 (VDDIO)
- net TMS: now reaches U6.13 (IO14)
- net TMS: now also R31.1
- net TCK: now reaches U6.16 (IO13)
- net TCK: now also R29.1
- net TDO: now reaches U6.23 (IO15)
- net TDO: now also R27.1
- net at U6.28 (IO17): now also R32.1
- net at R4.1: now also U2.1, U2.2 (-)
- net at R15.2, R4.2: now also U2.6 (-); no longer U2.5 (+)
- net at D3.1 (A1), F2.1: now also J4.1
- net at F2.2, R1.1: now also R3.1
- net at C4.2, C5.1, D1.3 (COM)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: now also U2.3 (+)
- net at R5.2, R7.1: now also U2.5 (+); no longer U2.6 (-)
- net TXEN: no longer names the net of U6.33 (IO21)
- net TXEN: now also U5.16 (TXEN)
- new net: D4.1 (A1), F1.1, J4.4
- new net: J1.R1 (TD+), R38.2, U5.21 (TXP)
- new net: J1.R6 (RD-), R42.2, U5.22 (RXN)
- new net: J1.L3, R44.1
- new net: C28.2, C29.2, U5.6 (VDDCR)
- new net: R33.2, U5.8 (RXD0/MODE0)
- new net: R27.2, U3.2 (TDO)
- new net: R29.2, U3.3 (TCK)
- new net: R30.2, U3.4 (TDI)
- new net: R31.2, U3.5 (TMS)
- new net: J1.R2 (TD-), R39.2, U5.20 (TXN)
- new net: J1.R3 (RD+), R41.2, U5.23 (RXP)
- new net: R37.1, U5.24 (RBIAS)
- new net: R34.2, U5.7 (RXD1/MODE1)
- new net: J1.L2, R45.1
- new net L1: J1.L1, R40.1, U5.2 (LED2/nINTSEL)
- new net L4: J1.L4, R43.2, U5.3 (LED1/REGOFF)
- new net RXER: R36.1, U5.10 (RXER/PHYAD0)
- new net TDI: R26.2, R30.1, U6.14 (IO12)
- no-connect marks 2 -> 1

Commit message: feat: Update to tanklevel v2 pcb
Parts:
- removed F2: 100mA, Fuse:Fuse_0603_1608Metric_Pad1.05x0.95mm_HandSolder, symbol Device:Fuse_Small
- removed U1: wuerthDebug6, awesome:wuerthDebug6, symbol awesome:wuerthDebug6
- removed U3: wuerthJTAG, awesome:wuerthJTAG, symbol awesome:wuerthJTAG
- added D5, D6: LED, LED_SMD:LED_0603_1608Metric_Pad1.05x0.95mm_HandSolder, symbol Device:LED
- added H1, H2: MountingHole, MountingHole:MountingHole_2.2mm_M2_DIN965, symbol Mechanical:MountingHole
- added R35, R46: 10K, Resistor_SMD:R_0603_1608Metric_Pad0.98x0.95mm_HandSolder, symbol Device:R
- added R8: 47R, Resistor_SMD:R_0603_1608Metric_Pad0.98x0.95mm_HandSolder, symbol Device:R
- added U8: wuerthDebug10, awesome:wuerth10, symbol awesome:wuerthDebug10
- C1, C13, C17, C19, C21, C24, C25, C4, C6: LCSC PN (none) -> C14663
- C12: LCSC PN (none) -> C15850
- C2, C9: LCSC PN (none) -> C28323
- C20, C29, C7: footprint Capacitor_SMD:C_0603_1608Metric_Pad1.08x0.95mm_HandSolder -> Capacitor_SMD:C_0805_2012Metric_Pad1.18x1.45mm_HandSolder; LCSC PN (none) -> C28323
- C22: footprint Capacitor_SMD:C_1210_3225Metric_Pad1.33x2.70mm_HandSolder -> Capacitor_SMD:C_1206_3216Metric_Pad1.33x1.80mm_HandSolder; LCSC PN (none) -> C51205
- C23: footprint Capacitor_SMD:C_1210_3225Metric_Pad1.33x2.70mm_HandSolder -> Capacitor_SMD:C_1206_3216Metric_Pad1.33x1.80mm_HandSolder; LCSC PN (none) -> C13585
- C26, C5: footprint Capacitor_SMD:C_0603_1608Metric_Pad1.08x0.95mm_HandSolder -> Capacitor_SMD:C_0805_2012Metric_Pad1.18x1.45mm_HandSolder; LCSC PN (none) -> C15850
- C27: value 10u -> 47u; footprint Capacitor_SMD:C_0603_1608Metric_Pad1.08x0.95mm_HandSolder -> Capacitor_SMD:C_1210_3225Metric_Pad1.33x2.70mm_HandSolder; LCSC PN (none) -> C77101
- C28: LCSC PN (none) -> C85979
- C3: LCSC PN (none) -> C1779
- C30: LCSC PN (none) -> C282065
- D1: LCSC PN (none) -> C7420333
- D2: LCSC PN (none) -> C8678
- D3: LCSC PN (none) -> C19077497; now not fitted; now left out of the parts list
- D4: LCSC PN (none) -> C19077514
- F1: LCSC PN (none) -> C151139
- FB2: footprint Capacitor_SMD:C_0603_1608Metric_Pad1.08x0.95mm_HandSolder -> Inductor_SMD:L_0603_1608Metric_Pad1.05x0.95mm_HandSolder; LCSC PN (none) -> C710376
- J1, J4, L1, PGAIN1, PZERO1, U4: now left out of the parts list
- R1: LCSC PN (none) -> C870446
- R12, R14, R32, R33, R34: value 33R -> 22R; LCSC PN (none) -> C138283
- R13, R18, R24, R25, R26, R28, R36, R4, R40, R43, R5, R6: LCSC PN (none) -> C140867
- R15, R7: LCSC PN (none) -> C137798
- R17: LCSC PN (none) -> C122970; now not fitted; now left out of the parts list
- R27, R29, R30, R31: LCSC PN (none) -> C122970
- R3: LCSC PN (none) -> C114623
- R37: LCSC PN (none) -> C245906
- R38, R39, R41, R42: value 50R -> 51R; LCSC PN (none) -> C23197
- R44, R45: LCSC PN (none) -> C22548
- U2: LCSC PN (none) -> C57639; now not fitted; now left out of the parts list
- U5: LCSC PN (none) -> C45223
- U6: LCSC PN (none) -> C701341
- U7: LCSC PN (none) -> C36310
Connections:
- net +3.3V: now also U8.3 (3V3)
- net ADC_IN: now also R8.2
- net BOOT0: now also U8.6 (BOOT0)
- net EN: now also U8.1 (EN)
- net GND: now also D5.1 (K), D6.1 (K), U8.2 (GND)
- net RXD: now also U8.5 (RXD)
- net TXD: now also U8.4 (TXD)
- net at U6.24 (IO2): now also R35.1
- net at U6.26 (IO4): now also R46.1
- net at D3.1 (A1), J4.1: now also R1.1, R3.1
- net at C4.2, C5.1, D1.3 (COM)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: now also R8.1
- net at R27.2: now also U8.7 (TDO)
- net at R29.2: now also U8.8 (TCK)
- net at R30.2: now also U8.9 (TDI)
- net at R31.2: now also U8.10 (TMS)
- new net: D6.2 (A), R46.2
- new net: D5.2 (A), R35.2
Other:
- moved on the sheet: R27, R29, R30, R31

Commit message: feat: Create fab output
Parts:
- C1, C13, C17, C19, C21, C24, C25, C28, C30, C4, C6: footprint Capacitor_SMD:C_0603_1608Metric_Pad1.08x0.95mm_HandSolder -> Capacitor_SMD:C_0603_1608Metric
- C12, C2, C20, C26, C29, C3, C5, C7, C9: footprint Capacitor_SMD:C_0805_2012Metric_Pad1.18x1.45mm_HandSolder -> Capacitor_SMD:C_0805_2012Metric
- C22, C23: footprint Capacitor_SMD:C_1206_3216Metric_Pad1.33x1.80mm_HandSolder -> Capacitor_SMD:C_1206_3216Metric
- C27: footprint Capacitor_SMD:C_1210_3225Metric_Pad1.33x2.70mm_HandSolder -> Capacitor_SMD:C_1210_3225Metric
- D5, D6: footprint LED_SMD:LED_0603_1608Metric_Pad1.05x0.95mm_HandSolder -> LED_SMD:LED_0603_1608Metric
- F1: footprint Fuse:Fuse_0603_1608Metric_Pad1.05x0.95mm_HandSolder -> Fuse:Fuse_0603_1608Metric
- FB2: footprint Inductor_SMD:L_0603_1608Metric_Pad1.05x0.95mm_HandSolder -> Inductor_SMD:L_0603_1608Metric
- R1: footprint Resistor_SMD:R_1206_3216Metric_Pad1.30x1.75mm_HandSolder -> Resistor_SMD:R_1206_3216Metric
- R12, R13, R14, R15, R17, R18, R24, R25, R26, R27, R28, R29, R3, R30, R31, R32, R33, R34, R35, R36, R37, R38, R39, R4, R40, R41, R42, R43, R44, R45, R46, R5, R6, R7, R8: footprint Resistor_SMD:R_0603_1608Metric_Pad0.98x0.95mm_HandSolder -> Resistor_SMD:R_0603_1608Metric
